File: hw/bizcamera.kicad_pcb (KiCad board)
At the start: 4 copper layers, 84.5 x 55 mm, 94 parts, among them J1 Camera, J2 Micro_SD_Card_Det1, J3 USB_IN, SW1 USB_BOOT, SW3 Shutter, U1 RP2350_60QFN, U2 SPX3819M5-L-1-8, U3 S25FS128SDSNFI101, U4 ESP-PSRAM64, U5 SPX3819M5-L-3-3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

Commit message: Directory update
Parts:
- BT1: footprint Battery:BatteryHolder_Keystone_3009_1x2450 -> Battery:BatteryHolder_Bulgin_BX0123_1xCR123
- C31, C32: footprint Capacitor_Tantalum_SMD:CP_EIA-6032-20_AVX-F_Pad2.25x2.35mm_HandSolder -> Capacitor_SMD:C_0603_1608Metric
- moved G*** 39.4 mm to (95.0, 71.8)
- moved REF** 37.5 mm to (105.4, 77.5)
- moved kibuzzard-68265FDC 32.0 mm to (140.4, 96.5), turned to -90 degrees
- moved C30 25.0 mm to (139.7, 101.0), turned to -90 degrees
- moved L2 24.0 mm to (137.5, 101.3), turned to 180 degrees
- moved U7 20.9 mm to (138.9, 103.8), turned to 0 degrees
- moved R19 18.9 mm to (140.1, 105.7), turned to 180 degrees
- moved BT1 18.5 mm to (124.5, 78.4)
- moved R6 18.0 mm to (140.8, 107.2), turned to 90 degrees
- moved kibuzzard-6825B58C 17.5 mm to (100.9, 82.2)
- moved C32 12.9 mm to (136.8, 106.7), turned to -90 degrees
- moved C31 11.2 mm to (138.3, 106.7), turned to -90 degrees
- moved kibuzzard-682743A4 0.23 mm to (144.2, 115.6)
Routing:
- net -BATT: track 149.1 -> 130.4 mm, vias 27 -> 26
- net +BATT: track 46.5 -> 34.9 mm
- net +3V3: track 50.5 -> 55.3 mm, vias 13 -> 8
- net Net-(U7-FB): track 3.29 -> 1.73 mm
- removed copper zone on F.Cu, net +3V3
